Commit message: updated to work in ros2 humble, including visualization of robot state in rviz

File: description/gazebo_control.xacro (robot description, xacro)
@@ -1,4 +1,17 @@
 <?xml version="1.0"?>
 <robot xmlns:xacro="http://www.ros.org/wiki/xacro">
+	<gazebo>
+		<plugin name='joint_state_publisher' filename='libgazebo_ros_joint_state_publisher.so'>
+			<ros>
+				<namespace>/</namespace>
+				<remapping>~/out:=joint_states</remapping>
+			</ros>
+			<update_rate>20</update_rate>
+			<joint_name>wheel1_joint</joint_name>
+			<joint_name>wheel2_joint</joint_name>
+			<joint_name>wheel3_joint</joint_name>
+			<joint_name>wheel4_joint</joint_name>
+		</plugin>
+	</gazebo>
 	<gazebo>
 		<plugin name="holonomic_control" filename="libgazebo_ros_planar_move.so">
@@ -7,5 +20,5 @@
       		<odometryFrame>odom</odometryFrame>
       		<odometryRate>20.0</odometryRate>
-      		<robotBaseFrame>base_link</robotBaseFrame>
+      		<robotBaseFrame>base_footprint</robotBaseFrame>
 			<publishTF>true</publishTF>
     	</plugin>

File: description/robot.urdf.xacro (robot description, xacro)
@@ -1,6 +1,6 @@
 <?xml version="1.0"?>
 <robot xmlns:xacro="http://www.ros.org/wiki/xacro"  name="robot">
-	<xacro:include filename="robot_core_highres.xacro"/>
-    <!--<xacro:include filename="robot_core.xacro"/>--> <!--Uncomment to use low res mode-->
+	<!--xacro:include filename="robot_core_highres.xacro"/-->
+    <xacro:include filename="robot_core.xacro"/> <!--Uncomment to use low res mode-->
     <xacro:include filename="gazebo_control.xacro"/>
 </robot>

File: description/robot_core.xacro (robot description, xacro)
@@ -14,4 +14,11 @@
 		<color rgba="0 0 0 1"/>
     </material>
+    <!-- BASE FOOTPRINT -->
+    <link name="base_footprint"/>
+    <joint name="base_joint" type="fixed">
+        <parent link="base_footprint"/>
+        <child link="base_link"/>
+        <origin xyz="0 0 0.08" rpy="0 0 0"/>  <!-- Height of wheel radius -->
+    </joint>
     <!-- BASE LINK -->
     <link name="base_link">
