Commit message: updates to cleanup urdf and make robot work with external test framework

File: description/robot_core.xacro (robot description, xacro)
@@ -32,5 +32,5 @@
 	<link name="chassis">
 		<visual>
-			<origin xyz="0 0 0.1"/>
+			<origin xyz="0 0 0.02"/>
 			<geometry>
 				<box size="0.5 0.5 0.03"/>
@@ -39,5 +39,5 @@
 		</visual>
 		<collision>
-			<origin xyz="0 0 0.1"/>
+			<origin xyz="0 0 0.02"/>
 			<geometry>
 				<box size="0.5 0.5 0.03"/>
@@ -55,5 +55,5 @@
 		<parent link="base_link"/>
 		<child link="wheel1_link"/>
-		<origin xyz="0 0.27 0.08" rpy="-${pi/2} 0 0"/>
+		<origin xyz="0 0.27 0.0" rpy="-${pi/2} 0 0"/>
 		<axis xyz="0 0 1"/>
 	</joint>
@@ -82,5 +82,5 @@
 		<parent link="base_link"/>
 		<child link="wheel2_link"/>
-		<origin xyz="0 -0.27 0.08" rpy="${pi/2} 0 0"/>
+		<origin xyz="0 -0.27 0.0" rpy="${pi/2} 0 0"/>
 		<axis xyz="0 0 -1"/>
 	</joint>
@@ -109,5 +109,5 @@
 		<parent link="base_link"/>
 		<child link="wheel3_link"/>
-		<origin xyz="0.27 0 0.08" rpy="${-pi/2} 0 ${-pi/2}"/>
+		<origin xyz="0.27 0 0.0" rpy="${-pi/2} 0 ${-pi/2}"/>
 		<axis xyz="0 0 1"/>
 	</joint>
@@ -136,5 +136,5 @@
 		<parent link="base_link"/>
 		<child link="wheel4_link"/>
-		<origin xyz="-0.27 0 0.08" rpy="${pi/2} 0 ${-pi/2}"/>
+		<origin xyz="-0.27 0 0.0" rpy="${pi/2} 0 ${-pi/2}"/>
 		<axis xyz="0 0 -1"/>
 	</joint>
